File: hydro-hat.kicad_sch (KiCad schematic)
At the start: 0 parts

Commit message: Basic connector placement, notes, todos
Parts:
- added C1: C, symbol Device:C
- added F1, F2, F4: Fuse, symbol Device:Fuse
- added H1, H2, H3, H4: MountingHole, symbol Mechanical:MountingHole
- added J1: RJ11 0-10V Dimming, symbol Connector:Conn_01x06_Socket
- added J2: Fan, Connector_Molex:Molex_KK-254_AE-6410-03A_1x03_P2.54mm_Vertical, symbol Connector:Conn_01x03_Pin
- added J3: Relay Board, symbol Connector:Conn_01x04_Socket
- added J4: Dual Rail PSU Input, symbol Connector:Conn_01x03_Socket
- added J5: Light State Pin, symbol Connector:Conn_01x02_Socket
- added J6: On Demand Light Switch, symbol Connector:Conn_01x02_Socket
- added J7: Raspberry_Pi_2_3, symbol Connector:Raspberry_Pi_2_3
- added J8, J9: eTape, symbol Connector_Generic_Shielded:Conn_01x04_Shielded
- added R1: 10k, symbol Device:R
- added R2, R3, R4: 430, symbol Device:R
Connections:
- new net: J6.2 (Pin_2), R1.2
- new net: F1.1, J4.3 (Pin_3)
- new net: J3.2 (Pin_2), R3.2
- new net: F4.1, J7.1 (3V3), J7.17 (3V3)
- new net: F2.1, J4.2 (Pin_2)
- new net: J3.1 (Pin_1), R4.1
- new net: J5.2 (Pin_2), R2.2
- new net +12V: F1.2, J2.1 (Pin_1)
- new net +3.3V: C1.1, F4.2, R1.1
- new net +5V: F2.2, J3.4 (Pin_4), J7.2 (5V), J7.4 (5V)
- new net GND: C1.2, J2.3 (Pin_3), J3.3 (Pin_3), J4.1 (Pin_1), J5.1 (Pin_1), J6.1 (Pin_1), J7.14 (GND), J7.20 (GND), J7.25 (GND), J7.30 (GND), J7.34 (GND), J7.39 (GND), J7.6 (GND), J7.9 (GND)
- new net Tacho: J2.2 (Pin_2)
- new net lightIsOn: R2.1
- new net relay1: R3.1
- new net relay2: R4.2
Other:
- note added: "10ms debounce"
- note added: "1: Reference + 2: Measure + 3: Measure - 4: Reference -"
- note added: "ADC resolution requirements Waterlevel with 50ml precision Tanks: - Sloped Box H: 30cm W: 38cm D: 76cm V: 63l - Big Tank: H: 60cm Dia: 45cm V: 60l - Paint Bucket: H: 20cm Dia:25cm V: 10l Worst case for resolution sloped box 300mm / 63l = 4,76 mm / l 50ml difference changes water level by 0.24mm 12" eTape has active length of 315mm 315mm / 0.24mm = 1313 ADC Steps Sensor starts from 0.4kR, not from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"
- note added: "Milone eTape"
- note added: "ToDo how much current do lights sink todo 3.3V logic level mosfet, high side switching"
- note added: "ToDo i²c ADC"
- note added: "Todo Differential Opamp, dual channel"
- note added: "Vmax = 10V Pmax = 0.5W"
- note added: "eTapes Used: 24" Ref: 4kR +-20% Measure: 0.4 - 4kR 12" Ref: 2kR +-20% Meausre: 0.4 - 2kR 8" Ref: 1.5kR +-20% Measure: 0.4 - 1.5kR Measure: 60R / cm"
- note added: "relay 1 pump relay 2 exhaust fan"
- note added: "todo can raspi be powered from this 5V port? todo 3.3v rail power rating"
- note added: "todo mosfet how to connect to raspi? connect tacho?"
- note added: "todo what shielded connector"

Commit message: Specified fuses, selected connectors, selected adc
- 3.3V, 5V fuse spec for raspi from pinout.xyz
- de9 connector for eTapes (shielded + cheap)
- ad7298 adc, easily available
Parts:
- removed J8, J9: eTape, symbol Connector_Generic_Shielded:Conn_01x04_Shielded
- added J10: eTape1, symbol Connector:DE9_Socket_MountingHoles
- added J11: eTape2, symbol Connector:DE9_Socket_MountingHoles
- added U1: AD7298, Package_CSP:LFCSP-20-1EP_4x4mm_P0.5mm_EP2.6x2.6mm_ThermalVias, symbol Analog_ADC:AD7298
- F2: value Fuse -> 3A
- F4: value Fuse -> 0.5A
Other:
- note added: "Todo wheatstone bridge + opamp"
- note added: "https://pinout.xyz/pinout/3v3_power"
- note removed: "ToDo i²c ADC"
- note removed: "Todo Differential Opamp, dual channel"
- note removed: "todo can raspi be powered from this 5V port? todo 3.3v rail power rating"
- note removed: "todo what shielded connector"

Commit message: notes about optocoupling
Other:
- note added: "todo optocoupler"
Changed lines of the file:
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@@
 	(generator_version "9.0")
 	(paper "A4")
+	(text "todo optocoupler"
+		(exclude_from_sim no)
+		(at 36.83 179.324 0)
+		(effects
+			(font
+				(size 1.27 1.27)
+			)
+		)
+	)
 	(text "Todo wheatstone bridge + opamp"
 		(exclude_from_sim no)
